Commit message: Update urdf to simulate the mouvements of the robot base

File: urdf/youbot.urdf (robot description, URDF)
Before this commit: robot youbot, 20 links, 19 joints
Links:
- added link virtual_link_xy
- added link virtual_link_yz
Joints:
- removed joint fixed
- added joint virtual_joint_x: type prismatic, parent world, child virtual_link_xy, axis 1 0 0, limit lower=-5 upper=5 effort=1 velocity=1
- added joint virtual_joint_y: type prismatic, parent virtual_link_xy, child virtual_link_yz, axis 0 1 0, limit lower=-5 upper=5 effort=1 velocity=1
- added joint virtual_joint_z: type continuous, parent virtual_link_yz, child base_footprint, origin xyz=0 0 0.1, axis 0 0 1
